File: traffic_control_system/Hardware/Controller_Board/Valve_Drive.kicad_sch (KiCad schematic)
At the start: 38 parts, among them J4 Screw_Terminal_01x12

Commit message: issue : 깃 커밋 히스토리 정리를 위한 원본 저장소의 브랜치 분리 작업[TRAFFIC-CONTROL6]
Parts:
- added J2: Screw_Terminal_01x11, symbol Connector:Screw_Terminal_01x11
- added R133, R134, R135, R136, R149, R150, R151, R152: 0R0F/0805, Resistor_SMD:R_0805_2012Metric, symbol Device:R
Connections:
- net GNDA: now also J2.3 (Pin_3), J2.6 (Pin_6), J2.9 (Pin_9)
- new net: J2.2 (Pin_2), R149.2
- new net: J2.5 (Pin_5), R150.2
- new net: J2.8 (Pin_8), R151.2
- new net: J2.11 (Pin_11), R152.2
- new net +24V: J2.1 (Pin_1), J2.10 (Pin_10), J2.4 (Pin_4), J2.7 (Pin_7)
- new net cylinder_pos_sening/valve_pos1: R133.2
- new net cylinder_pos_sening/valve_pos2: R134.2
- new net cylinder_pos_sening/valve_pos3: R135.2
- new net cylinder_pos_sening/valve_pos4: R136.2
- new net cylinder_pos_sening/valvea_pos1-: R149.1
- new net cylinder_pos_sening/valvea_pos2-: R150.1
- new net cylinder_pos_sening/valvea_pos3-: R151.1
- new net cylinder_pos_sening/valvea_pos4-: R152.1
- new net valve_pos1_o: R133.1
- new net valve_pos2_o: R134.1
- new net valve_pos3_o: R135.1
- new net valve_pos4_o: R136.1
- no-connect marks 1 -> 0
Other:
- added sheet cylinder_pos_sening (cylinder_pos_sening.kicad_sch)
- moved on the sheet: J4, R101, R102, R103, R104, R33, R34, R35, R36, R37, R38, R39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
